File: cad/magnswi/magnswi.kicad_pcb (KiCad board)
At the start: 2 copper layers, 22 x 63.5 mm, 16 parts, among them J1 Conn_02x04_Top_Bottom, SW1 SW_DPST_x2, SW2 SW_Reed, U1 nrf528324_mod_mkbno2

Commit message: darn aliexpress
Parts:
- C2: footprint Capacitor_SMD:C_0603_1608Metric -> Capacitor_SMD:C_0402_1005Metric
- R1, R2: value 20k -> 5k
- R3: value 330 -> 240
- R4: value 330 -> 300
- R6: value 1M -> 100k
- U1: value nrf528324_mod_mkbno2 -> nrf52832_mod_holyiot17095; footprint pelle:mkbno2 -> pelle:holyiot17095
- moved U1 9.03 mm to (6.25, -51.2)
Connections:
- J1 pad 1: UART_RX -> (no net)
- J1 pad 2: UART_TX -> (no net)
- J1 pad 3: SWDIO -> (no net)
- J1 pad 4: SWDCLK -> (no net)
- R2 pad 1: BATT_SPL_EN -> (no net)
- R3 pad 1: LED_G -> (no net)
- R4 pad 1: LED_R -> (no net)
- SW2 pad 2: SW_MAGNET_EN -> (no net)
- U1 pad 10: GND -> (no net)
- U1 pad 11: SW_MAGNET_EN -> (no net)
- U1 pad 12: SW_MAGNET -> (no net)
- U1 pad 13: BATT_SPL -> (no net)
- U1 pad 14: BATT_SPL_EN -> (no net)
- U1 pad 15: SW_TAMPER_EN -> (no net)
- U1 pad 9: +3V0 -> (no net)
Routing:
- net (no net): track 0.00 -> 272.6 mm, vias 2 -> 9
- net UART_RX: track 52.4 -> 0.00 mm
- net UART_TX: track 48.5 -> 0.00 mm
- net SWDIO: track 44.9 -> 0.00 mm
- net SWDCLK: track 42.4 -> 0.00 mm
- net SW_MAGNET_EN: track 38.7 -> 0.00 mm
- net LED_R: track 21.3 -> 0.00 mm, vias 2 -> 0
- net LED_G: track 19.8 -> 0.00 mm, vias 2 -> 0
- net BATT_SPL_EN: track 4.52 -> 0.00 mm
- net GND: vias 49 -> 46
